File: MotorDriver/MotorDriver.kicad_pcb (KiCad board)
At the start: 2 copper layers, 6 parts, among them P101 CONTROL, P102 MOT, P103 Vm, U101 ZXBM5210

Commit message: Clean up motor driver board.
Parts:
- added G***: LOGO, gl:ce-logo, B.Cu at (181.4, 104.1)
- moved C102 0.25 mm to (181.4, 96.5)
Other:
- board outline added: 14.6 x 14.2 mm
- board text added: "+"
- board text added: "F"
- board text added: "G"
- board text added: "GoGoGo!"
- board text added: "MOT"
- board text added: "R"
- board text added: "V"
